File: Schematic/Anemometer/Anemometer.kicad_sch (KiCad schematic)
At the start: 9 parts, among them J1 Battery, J2 Screen, J3 CG_Anem, U1 TP4065_ChargeModule, U2 MCP1700x-330xxTO, U3 WeMos_D1_mini

Commit message: Added PCB 3D model
Connections:
- net GND: now also J2.3 (Pin_3), J3.3 (Pin_3); no longer J2.2 (Pin_2), J3.2 (Pin_2)
- net at C2.1, U2.3 (VO), U3.8 (3V3): now also J2.4 (Pin_4), J3.4 (Pin_4); no longer J2.1 (Pin_1), J3.1 (Pin_1)
- net at U1.4 (+BAT): now also J1.2 (Pin_2); no longer J1.1 (Pin_1)
- net at U1.5 (-BAT): now also J1.1 (Pin_1); no longer J1.2 (Pin_2)
- new net: J2.1 (Pin_1), J3.1 (Pin_1), U3.13 (SDA/D2)
- new net: J2.2 (Pin_2), J3.2 (Pin_2), U3.14 (SCL/D1)
Other:
- moved on the sheet: J1
Changed lines of the file:
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@@
   (junction (at 85.09 36.83) (diameter 0) (color 0 0 0 0)
   )
+  (junction (at 123.19 66.04) (diameter 0) (color 0 0 0 0)
+  )
   (junction (at 107.95 36.83) (diameter 0) (color 0 0 0 0)
   )
-  (junction (at 123.19 66.04) (diameter 0) (color 0 0 0 0)
+  (junction (at 128.27 60.96) (diameter 0) (color 0 0 0 0)
   )
   (junction (at 125.73 63.5) (diameter 0) (color 0 0 0 0)
@@
   (junction (at 92.71 44.45) (diameter 0) (color 0 0 0 0)
   )
-  (junction (at 128.27 60.96) (diameter 0) (color 0 0 0 0)
-  )
   (wire (pts (xy 66.04 34.29) (xy 71.12 34.29))
     (stroke (width 0) (type default) (color 0 0 0 0))
   )
-  (wire (pts (xy 128.27 77.47) (xy 128.27 60.96))
-    (stroke (width 0) (type default) (color 0 0 0 0))
-  )
   (wire (pts (xy 107.95 53.34) (xy 107.95 36.83))
     (stroke (width 0) (type default) (color 0 0 0 0))
   )
-  (wire (pts (xy 130.81 80.01) (xy 125.73 80.01))
-    (stroke (width 0) (type default) (color 0 0 0 0))
-  )
   (wire (pts (xy 107.95 36.83) (xy 128.27 36.83))
     (stroke (width 0) (type default) (color 0 0 0 0))
@@
     (stroke (width 0) (type default) (color 0 0 0 0))
   )
+  (wire (pts (xy 128.27 60.96) (xy 128.27 77.47))
+    (stroke (width 0) (type default) (color 0 0 0 0))
+  )
   (wire (pts (xy 69.85 36.83) (xy 69.85 48.26))
     (stroke (width 0) (type default) (color 0 0 0 0))
@@
     (stroke (width 0) (type default) (color 0 0 0 0))
   )
+  (wire (pts (xy 128.27 60.96) (xy 130.81 60.96))
+    (stroke (width 0) (type default) (color 0 0 0 0))
+  )
   (wire (pts (xy 130.81 85.09) (xy 120.65 85.09))
     (stroke (width 0) (type default) (color 0 0 0 0))
   )
-  (wire (pts (xy 125.73 80.01) (xy 125.73 63.5))
-    (stroke (width 0) (type default) (color 0 0 0 0))
-  )
   (wire (pts (xy 62.23 36.83) (xy 69.85 36.83))
     (stroke (width 0) (type default) (color 0 0 0 0))
@@
     (stroke (width 0) (type default) (color 0 0 0 0))
   )
+  (wire (pts (xy 123.19 82.55) (xy 123.19 66.04))
+    (stroke (width 0) (type default) (color 0 0 0 0))
+  )
+  (wire (pts (xy 85.09 44.45) (xy 92.71 44.45))
+    (stroke (width 0) (type default) (color 0 0 0 0))
+  )
+  (wire (pts (xy 123.19 82.55) (xy 130.81 82.55))
+    (stroke (width 0) (type default) (color 0 0 0 0))
+  )
+  (wire (pts (xy 128.27 36.83) (xy 128.27 60.96))
+    (stroke (width 0) (type default) (color 0 0 0 0))
+  )
+  (wire (pts (xy 128.27 77.47) (xy 130.81 77.47))
+    (stroke (width 0) (type default) (color 0 0 0 0))
+  )
+  (wire (pts (xy 123.19 66.04) (xy 130.81 66.04))
+    (stroke (width 0) (type default) (color 0 0 0 0))
+  )
+  (wire (pts (xy 100.33 44.45) (xy 125.73 44.45))
+    (stroke (width 0) (type default) (color 0 0 0 0))
+  )
+  (wire (pts (xy 85.09 33.02) (xy 115.57 33.02))
+    (stroke (width 0) (type default) (color 0 0 0 0))
+  )
+  (wire (pts (xy 107.95 36.83) (xy 100.33 36.83))
+    (stroke (width 0) (type default) (color 0 0 0 0))
+  )
+  (wire (pts (xy 120.65 85.09) (xy 120.65 68.58))
+    (stroke (width 0) (type default) (color 0 0 0 0))
+  )
+  (wire (pts (xy 62.23 45.72) (xy 62.23 53.34))
+    (stroke (width 0) (type default) (color 0 0 0 0))
+  )
+  (wire (pts (xy 67.31 41.91) (xy 67.31 48.26))
+    (stroke (width 0) (type default) (color 0 0 0 0))
+  )
+  (wire (pts (xy 62.23 34.29) (xy 66.04 34.29))
+    (stroke (width 0) (type default) (color 0 0 0 0))
+  )
+  (wire (pts (xy 125.73 63.5) (xy 125.73 80.01))
+    (stroke (width 0) (type default) (color 0 0 0 0))
+  )
+  (wire (pts (xy 81.28 36.83) (xy 85.09 36.83))
+    (stroke (width 0) (type default) (color 0 0 0 0))
+  )
   (wire (pts (xy 125.73 63.5) (xy 130.81 63.5))
     (stroke (width 0) (type default) (color 0 0 0 0))
   )
-  (wire (pts (xy 123.19 82.55) (xy 123.19 66.04))
-    (stroke (width 0) (type default) (color 0 0 0 0))
-  )
-  (wire (pts (xy 85.09 44.45) (xy 92.71 44.45))
-    (stroke (width 0) (type default) (color 0 0 0 0))
-  )
-  (wire (pts (xy 128.27 36.83) (xy 128.27 60.96))
-    (stroke (width 0) (type default) (color 0 0 0 0))
-  )
-  (wire (pts (xy 128.27 60.96) (xy 130.81 60.96))
-    (stroke (width 0) (type default) (color 0 0 0 0))
-  )
-  (wire (pts (xy 100.33 44.45) (xy 125.73 44.45))
-    (stroke (width 0) (type default) (color 0 0 0 0))
-  )
-  (wire (pts (xy 85.09 33.02) (xy 115.57 33.02))
-    (stroke (width 0) (type default) (color 0 0 0 0))
-  )
-  (wire (pts (xy 130.81 82.55) (xy 123.19 82.55))
-    (stroke (width 0) (type default) (color 0 0 0 0))
-  )
-  (wire (pts (xy 107.95 36.83) (xy 100.33 36.83))
-    (stroke (width 0) (type default) (color 0 0 0 0))
-  )
-  (wire (pts (xy 120.65 85.09) (xy 120.65 68.58))
-    (stroke (width 0) (type default) (color 0 0 0 0))
-  )
-  (wire (pts (xy 62.23 45.72) (xy 62.23 53.34))
-    (stroke (width 0) (type default) (color 0 0 0 0))
-  )
-  (wire (pts (xy 67.31 41.91) (xy 67.31 48.26))
-    (stroke (width 0) (type default) (color 0 0 0 0))
-  )
-  (wire (pts (xy 62.23 34.29) (xy 66.04 34.29))
-    (stroke (width 0) (type default) (color 0 0 0 0))
-  )
-  (wire (pts (xy 81.28 36.83) (xy 85.09 36.83))
-    (stroke (width 0) (type default) (color 0 0 0 0))
-  )
-  (wire (pts (xy 130.81 77.47) (xy 128.27 77.47))
-    (stroke (width 0) (type default) (color 0 0 0 0))
-  )
-  (wire (pts (xy 123.19 66.04) (xy 130.81 66.04))
-    (stroke (width 0) (type default) (color 0 0 0 0))
-  )
-  (symbol (lib_id "Connector_Generic:Conn_01x04") (at 135.89 63.5 0) (unit 1)
-    (in_bom yes) (on_board yes) (fields_autoplaced)
-    (property "Reference" "J2" (id 0) (at 138.43 63.4999 0)
-      (effects (font (size 1.27 1.27)) (justify left))
-    )
-    (property "Value" "Screen" (id 1) (at 138.43 66.0399 0)
-      (effects (font (size 1.27 1.27)) (justify left))
-    )
-    (property "Footprint" "Connector_PinSocket_2.54mm:PinSocket_1x04_P2.54mm_Vertical" (id 2) (at 135.89 63.5 0)
-      (effects (font (size 1.27 1.27)) hide)
-    )
-    (property "Datasheet" "~" (id 3) (at 135.89 63.5 0)
+  (wire (pts (xy 125.73 80.01) (xy 130.81 80.01))
+    (stroke (width 0) (type default) (color 0 0 0 0))
+  )
+  (symbol (lib_id "Connector_Generic:Conn_01x04") (at 135.89 66.04 0) (mirror x) (unit 1)
+    (in_bom yes) (on_board yes) (fields_autoplaced)
+    (property "Reference" "J2" (id 0) (at 135.89 54.61 0))
+    (property "Value" "Screen" (id 1) (at 135.89 57.15 0))
+    (property "Footprint" "Connector_PinSocket_2.54mm:PinSocket_1x04_P2.54mm_Vertical" (id 2) (at 135.89 66.04 0)
+      (effects (font (size 1.27 1.27)) hide)
+    )
+    (property "Datasheet" "~" (id 3) (at 135.89 66.04 0)
       (effects (font (size 1.27 1.27)) hide)
     )
@@
     (pin "2")
   )
-  (symbol (lib_id "Connector_Generic:Conn_01x04") (at 135.89 80.01 0) (unit 1)
-    (in_bom yes) (on_board yes) (fields_autoplaced)
-    (property "Reference" "J3" (id 0) (at 138.43 80.0099 0)
-      (effects (font (size 1.27 1.27)) (justify left))
-    )
-    (property "Value" "CG_Anem" (id 1) (at 138.43 82.5499 0)
-      (effects (font (size 1.27 1.27)) (justify left))
-    )
-    (property "Footprint" "Connector_JST:JST_EH_S4B-EH_1x04_P2.50mm_Horizontal" (id 2) (at 135.89 80.01 0)
-      (effects (font (size 1.27 1.27)) hide)
-    )
-    (property "Datasheet" "~" (id 3) (at 135.89 80.01 0)
+  (symbol (lib_id "Connector_Generic:Conn_01x04") (at 135.89 82.55 0) (mirror x) (unit 1)
+    (in_bom yes) (on_board yes) (fields_autoplaced)
+    (property "Reference" "J3" (id 0) (at 135.89 71.12 0))
+    (property "Value" "CG_Anem" (id 1) (at 135.89 73.66 0))
+    (property "Footprint" "Connector_JST:JST_EH_S4B-EH_1x04_P2.50mm_Horizontal" (id 2) (at 135.89 82.55 0)
+      (effects (font (size 1.27 1.27)) hide)
+    )
+    (property "Datasheet" "~" (id 3) (at 135.89 82.55 0)
       (effects (font (size 1.27 1.27)) hide)
     )
@@
     (pin "3")
   )
-  (symbol (lib_id "Connector_Generic:Conn_01x02") (at 69.85 53.34 270) (unit 1)
+  (symbol (lib_id "Connector_Generic:Conn_01x02") (at 67.31 53.34 90) (mirror x) (unit 1)
     (in_bom yes) (on_board yes) (fields_autoplaced)
     (property "Reference" "J1" (id 0) (at 72.39 52.0699 90)
-      (effects (font (size 1.27 1.27)) (justify left))
+      (effects (font (size 1.27 1.27)) (justify right))
     )
     (property "Value" "Battery" (id 1) (at 72.39 54.6099 90)
-      (effects (font (size 1.27 1.27)) (justify left))
-    )
-    (property "Footprint" "Connector_JST:JST_EH_S2B-EH_1x02_P2.50mm_Horizontal" (id 2) (at 69.85 53.34 0)
-      (effects (font (size 1.27 1.27)) hide)
-    )
-    (property "Datasheet" "~" (id 3) (at 69.85 53.34 0)
-      (effects (font (size 1.27 1.27)) hide)
-    )
+      (effects (font (size 1.27 1.27)) (justify right))
+    )
+    (property "Footprint" "Connector_JST:JST_EH_S2B-EH_1x02_P2.50mm_Horizontal" (id 2) (at 67.31 53.34 0)
+      (effects (font (size 1.27 1.27)) hide)
+    )
+    (property "Datasheet" "~" (id 3) (at 67.31 53.34 0)
+      (effects (font (size 1.27 1.27)) hide)
+    )
